File: 05-Layout/nowae011/nowae011-0/nowae011.kicad_pcb (KiCad board)
At the start: 2 copper layers, 26.7 x 18.4 mm, 15 parts, among them P1 VIN, P2 VOUT, U1 ST1S14PHR

Commit message: Updated pcb (nowae011-0)
Parts:
- moved P2 1.27 mm to (24.1, -9.53)
- moved C4 1.21 mm to (17.8, -13.8)
- moved L1 1.21 mm to (17.8, -4.95)
- moved R1 1.08 mm to (13.5, -12.7)
- moved R2 1.08 mm to (13.5, -7.62)
- moved R3 1.08 mm to (13.5, -10.2)
- moved R4 1.08 mm to (13.5, -15.4)
- moved U1 0.89 mm to (9.27, -8.89)
- moved DL1 0.76 mm to (12.3, -15.4)
- moved C1 0.38 mm to (7.87, -14.7)
- moved C2 0.38 mm to (4.57, -8.26)
- moved C3 0.38 mm to (9.78, -5.46)
- moved D1 0.38 mm to (8.51, -2.79)
- moved G*** 0.38 mm to (13.0, -15.9)
Routing:
- net +5V: track 19.8 -> 14.0 mm
- net Net-(P2-Pad2): track 2.14 -> 0.00 mm
- net GND: track 19.0 -> 17.8 mm
Other:
- board size 26.7 x 18.4 mm -> 25.4 x 18.4 mm

Commit message: WiP: placement silkscreen (nowae011-0)
Other:
- board text added: "+24V"
- board text added: "+5V"
- board text added: "GND"
Changed lines of the file:
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@@
   (general
     (thickness 1.6)
-    (drawings 26)
+    (drawings 31)
     (tracks 52)
     (zones 0)
@@
     (34 B.Paste user hide)
     (35 F.Paste user hide)
-    (36 B.SilkS user hide)
+    (36 B.SilkS user)
     (37 F.SilkS user)
     (38 B.Mask user hide)
@@
       (xy 2.71208 1.245776)) (layer B.SilkS) (width 0.01))
   )
+  (gr_text +5V (at 20.32 -12.065) (layer B.SilkS)
+    (effects (font (size 1 1) (thickness 0.15)) (justify mirror))
+  )
+  (gr_text GND (at 20.32 -6.985) (layer B.SilkS)
+    (effects (font (size 1 1) (thickness 0.15)) (justify mirror))
+  )
+  (gr_text GND (at 5.715 -6.985) (layer B.SilkS)
+    (effects (font (size 1 1) (thickness 0.15)) (justify mirror))
+  )
+  (gr_text +24V (at 5.715 -12.065) (layer B.SilkS)
+    (effects (font (size 1 1) (thickness 0.15)) (justify mirror))
+  )
+  (gr_text +5V (at 12.7 -19.05) (layer F.SilkS)
+    (effects (font (size 1 1) (thickness 0.15)))
+  )
   (dimension 18.415 (width 0.3) (layer Dwgs.User)
