File: 05-Layout/nowae016/nowae016-0/nowae016.kicad_pcb (KiCad board)
At the start: 2 copper layers, 60 x 68.5 mm, 53 parts, among them P1 12VIN, P2 BATT1, P3 12VOUT1, P4 12VOUT2, P5 BATT2, Q1 BCW66GLT, U1 BQ24040DSQT, U2 TPS61087DRCR

Commit message: WiP: layout (nowae016-0)
Parts:
- removed the REF** at (3.50, -3.50)
- removed the REF** at (56.5, -3.50)
- REF** (x2): value HOLE-M2.5 -> SCREW-M2.5; footprint MECHANICAL:HOLE-M2.5 -> MECHANICAL:SCREW-M2.5
- moved G*** 70.5 mm to (51.0, 16.5)
- moved G*** 70.0 mm to (53.5, 20.0)
- moved G*** 70.0 mm to (53.5, 25.5)
- moved C1 68.5 mm to (12.2, 10.3)
- moved C10 68.5 mm to (31.2, 19.9)
- moved C11 68.5 mm to (27.2, 23.3)
- moved C12 68.5 mm to (29.2, 23.3)
- moved C2 68.5 mm to (17.4, 10.3)
- moved C3 68.5 mm to (13.6, 18.7)
- moved C4 68.5 mm to (13.6, 22.1)
- moved C5 68.5 mm to (15.2, 22.1)
- moved C6 68.5 mm to (16.6, 22.1)
- moved C7 68.5 mm to (16.6, 25.7)
- moved C8 68.5 mm to (27.2, 19.9)
- moved C9 68.5 mm to (29.2, 19.9)
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Routing:
- net +VBAT: track 58.2 -> 56.4 mm
- net /~CHG: track 65.5 -> 64.3 mm
- net +12V: track 18.7 -> 18.0 mm
Other:
- board size 60 x 68.5 mm -> 60 x 30 mm

Commit message: WiP: schematic (nowae016-0)
Routing:
- net GND: track 44.5 -> 47.5 mm
Changed lines of the file:
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@@
     (thickness 1.6)
     (drawings 41)
-    (tracks 185)
+    (tracks 187)
     (zones 0)
     (modules 51)
@@
   )
   (setup
-    (last_trace_width 0.25)
+    (last_trace_width 0.5)
     (user_trace_width 0.2)
     (user_trace_width 0.25)
@@
   (segment (start 46.45 24.5) (end 46.45 25.85) (width 0.25) (layer F.Cu) (net 1))
   (via (at 46.45 25.85) (size 0.6) (drill 0.3) (layers F.Cu B.Cu) (net 1))
+  (segment (start 19.2 22.675) (end 19.2 21.525) (width 0.5) (layer B.Cu) (net 1))
+  (segment (start 18.25 22.1) (end 20.15 22.1) (width 0.5) (layer B.Cu) (net 1))
   (segment (start 41.7 24.5) (end 43.55 24.5) (width 0.25) (layer F.Cu) (net 2))
   (segment (start 9.8 14.75) (end 9.8 14.5) (width 0.2) (layer F.Cu) (net 3))
