File: 05-Layout/NOWAE031-0/01-CCR_sch.kicad_sch (KiCad schematic)
At the start: 80 parts

Commit message: WiP: schematic (NOWAE031-0)
Parts:
- added C?: 22u, symbol nowae-capacitor:CAPACITOR_POL
- added C?: 4u7, symbol nowae-capacitor:CAPACITOR
- added D?: BAV21W-E3-08, DIODE:DIODE-SOD123, symbol nowae-diode:BAV21W-E3-08
- added D?: TS4148-RYG, DIODE:DIODE-0805, symbol nowae-diode:TS4148-RYG
- added DZ?: BZX384-C18,115, DIODE:DIODE-SOD323, symbol nowae-diode:BZX384-C18,115
- added Q?: BCX55-16,115, SOT:SOT89-3, symbol nowae-transistor:BCX55-16,115
- added R?: 33k, symbol nowae-resistor:RESISTOR
Connections:
- net AUX_ZCD: now also D?.1 (A)
- net GND: now also C?.2, C?.2, DZ?.1 (A)
- net VCC: now also C?.1, D?.2 (K)
- new net: DZ?.2 (K), Q?.1 (B), R?.1
- new net: D?.1 (A), Q?.2 (E), Q?.4 (E)
- new net: C?.1, D?.2 (K), Q?.3 (C), R?.2
Other:
- moved on the sheet: C?, D?, DZ?, F?, L?, P?, Q?, R?, T?, U, U?, VR?
